File: piPod_dev_board.sch (KiCad schematic (older format))
At the start: 25 parts, among them J1 USB_C_Receptacle_USB2.0, J2 Micro_SD_Card_Det_Hirose_DM3AT, Q1 DMG9926UDM, Q2 AO3401A, U1 AP9101CK, U2 MCP73828, U3 RP400N501A

Commit message: Redo power supply, switch to STM32 for SMC
Parts:
- removed A2: ARDUINO_PRO_MINI, Gigahawk:ARDUINO_PRO_MINI_THT, symbol gigahawk:ARDUINO_PRO_MINI
- removed D1, D2, D3, D4: PMEG2010AEH, Diode_SMD:D_SOD-123F, symbol Diode:PMEG2010AEH
- removed Q2: AO3401A, Package_TO_SOT_SMD:SOT-23, symbol Transistor_FET:AO3401A
- removed U2: MCP73828, Package_SO:MSOP-8_3x3mm_P0.65mm, symbol gigahawk:MCP73828
- removed U3: RP400N501A, Package_TO_SOT_SMD:SOT-23-5, symbol gigahawk:RP400N501A
- added C10, C7, C8: 100n, Capacitor_SMD:C_0805_2012Metric, symbol Device:CP1_Small
- added C9: 1u, Capacitor_SMD:C_0805_2012Metric, symbol Device:CP1_Small
- added D1: LEDB, symbol Device:LED
- added D2: LEDG, symbol Device:LED
- added D3: LEDR, symbol Device:LED
- added R10, R9: 10k, Resistor_SMD:R_0805_2012Metric, symbol Device:R_Small
- added R5: 300R, Resistor_SMD:R_0805_2012Metric, symbol Device:R_Small
- added R6: 2k, Resistor_SMD:R_0805_2012Metric, symbol Device:R_Small
- added R7: 1k54, Resistor_SMD:R_0805_2012Metric, symbol Device:R_Small
- added R8: 69k8, Resistor_SMD:R_0805_2012Metric, symbol Device:R_Small
- added U2: MCP73833-MSOP, Package_SO:MSOP-10_3x3mm_P0.5mm, symbol gigahawk:MCP73833-MSOP
- added U3: IPOD4_CW, Gigahawk:SFV8R2STE1HLF, symbol gigahawk:IPOD4_CW
- added U4: STM32L051C8Tx, Package_QFP:LQFP-48_7x7mm_P0.5mm, symbol MCU_ST_STM32L0:STM32L051C8Tx
- C2, C3, C4: value 10u -> 4u7
- C5: value 10u -> 100n
- L1: value L_Small -> 27n
- R3: value 100k -> 140R
- R4: value 100m -> 290R
Connections:
- net +3V3: now also C4.1, C5.1, L1.1, C7.1, C8.1, R10.1, R9.1, U3.1 (VCC), U4.24 (VDD), U4.36 (VDDIO2), U4.48 (VDD); no longer A1.1 (3V3), A1.17 (3V3), A1.PP8 (3V3)
- net +BATT: now also U2.10 (VBAT), U2.9 (VBAT)
- net GND: now also C10.2, C7.2, C8.2, C9.2, R6.1, R8.1, U2.5 (VSS), U3.8 (GND), U4.23 (VSS), U4.35 (VSS), U4.47 (VSS), U4.8 (VSSA)
- net THERM: now also R7.1, R8.2
- net VBUS: now also C2.1, D1.2 (A), D2.2 (A), D3.2 (A), U2.1 (VDD), U2.2 (VDD)
- net I2C_SDA: now reaches A1.3 (GPIO2/SDA)
- net I2C_SDA: now also U4.22 (PB11), U4.43 (PB7)
- net I2C_SCL: now reaches A1.5 (GPIO3/SCL)
- net I2C_SCL: now also U4.21 (PB10), U4.42 (PB6)
- net at R3.2: now also D1.1 (K)
- net at R4.1: now also U2.4 (STAT2)
- net +3.3VA: now reaches L1.2
- net +3.3VA: now also C10.1, C9.1, U4.9 (VDDA)
- net +1V8: no longer names the net of A1.PP9 (1V8)
- removed net +5V: A1.2 (5V), A1.4 (5V), C5.1
- new net: R10.2, U3.3 (EN2)
- new net: R9.2, U3.7 (EN1)
- new net: R3.1, U2.3 (STAT1)
- new net: R6.2, U2.6 (PROG)
- new net: R5.1, U2.7 (~PG)
- new net: R7.2, U2.8 (THERM)
- new net: D2.1 (K), R4.2
- new net: D3.1 (K), R5.2
- new net CW_CLK: U3.2 (CLK), U4.15 (PA5)
- new net CW_MOSI: U3.6 (MOSI), U4.17 (PA7)
- no-connect marks 6 -> 12
Other:
- note added: "Charge current \n= 1000mA*1kOhm/R_PROG"
- note added: "I2C1 as TCA8418 emulator\nI2C2 as SMC"
- note added: "Pi Zero can be safely powered off 3.3V if not using USB"
- note added: "Pi acts as I2C Master\n"
- note added: "Sample values from datasheet, \niPod battery thermistor parameters unknown"
- moved on the sheet: A1A

Commit message: Switch RPi footprint to THT
Parts:
- A1: footprint Gigahawk:RASPI_ZERO_1_3_SMT_LOW_PROFILE -> Gigahawk:RASPI_ZERO_1_3_THT
Changed lines of the file:
@@
 F 0 "A1" H 3550 700 50  0000 C CNN
 F 1 "RASPBERRY_PI_ZERO_SMT" H 4950 -1350 50  0000 C CNN
-F 2 "Gigahawk:RASPI_ZERO_1_3_SMT_LOW_PROFILE" H 4050 1000 50  0001 C CNN
+F 2 "Gigahawk:RASPI_ZERO_1_3_THT" H 4050 1000 50  0001 C CNN
 F 3 "" H 4050 1000 50  0001 C CNN
 	1    4100 950
@@
 F 0 "A1" H 1183 1865 50  0000 C CNN
 F 1 "RASPBERRY_PI_ZERO_SMT" H 1183 1774 50  0000 C CNN
-F 2 "Gigahawk:RASPI_ZERO_1_3_SMT_LOW_PROFILE" H 1200 1750 50  0001 C CNN
+F 2 "Gigahawk:RASPI_ZERO_1_3_THT" H 1200 1750 50  0001 C CNN
 F 3 "" H 1200 1750 50  0001 C CNN
 	2    1250 1700
@@
 F 0 "A1" H 1183 2415 50  0000 C CNN
 F 1 "RASPBERRY_PI_ZERO_SMT" H 1183 2324 50  0000 C CNN
-F 2 "Gigahawk:RASPI_ZERO_1_3_SMT_LOW_PROFILE" H 1200 2300 50  0001 C CNN
+F 2 "Gigahawk:RASPI_ZERO_1_3_THT" H 1200 2300 50  0001 C CNN
 F 3 "" H 1200 2300 50  0001 C CNN
 	3    1250 2250
@@
 F 0 "A1" H 8700 1050 50  0000 C CNN
 F 1 "RASPBERRY_PI_ZERO_SMT" H 9800 -350 50  0000 C CNN
-F 2 "Gigahawk:RASPI_ZERO_1_3_SMT_LOW_PROFILE" H 9050 1300 50  0001 C CNN
+F 2 "Gigahawk:RASPI_ZERO_1_3_THT" H 9050 1300 50  0001 C CNN
 F 3 "" H 9050 1300 50  0001 C CNN
 	4    9100 1250
